Commit message: Added Carriage STL for prismatic joints

File: urdf/aplotter.urdf (robot description, URDF)
Before this commit: robot aplotter, 5 links, 4 joints
Links:
- link leftPLink: geometry visual mesh filename=package://aplotter_ros2/urdf/carriage.stl
- link rightPLink: geometry visual mesh filename=package://aplotter_ros2/urdf/carriage.stl
Joints:
- joint leftPJoint: origin xyz=0 0 0 rpy=0 0 0 -> xyz=0 41.356 61 rpy=0 0 0
- joint rightPJoint: origin xyz=0 0 0 rpy=0 0 0 -> xyz=0 41.356 61 rpy=0 0 0

Commit message: Seperated arms and added forward kine

File: urdf/aplotter.urdf (robot description, URDF)
Before this commit: robot aplotter, 5 links, 4 joints
Links:
- link leftLink: geometry visual mesh filename=package://aplotter_ros2/urdf/larm.stl
- link rightLink: geometry visual mesh filename=package://aplotter_ros2/urdf/rarm.stl
Joints:
- joint leftJoint: axis 0 0 -1 -> 0 0 1
- joint leftPJoint: axis -1 0 0 -> 1 0 0
- joint rightJoint: axis 0 0 -1 -> 0 0 1; origin xyz=0 0 0 rpy=0 0 0 -> xyz=0 0 0 rpy=0 0 -0.12524034
- joint rightPJoint: axis -1 0 0 -> 1 0 0

Commit message: Working Inverse Kinematics with documentation

File: urdf/aplotter.urdf (robot description, URDF)
Before this commit: robot aplotter, 5 links, 4 joints
Joints:
- joint leftPJoint: origin xyz=0 41.356 61 rpy=0 0 0 -> xyz=0 41.356 71.042 rpy=0 0 0
- joint rightPJoint: origin xyz=0 41.356 61 rpy=0 0 0 -> xyz=0 41.356 71.042 rpy=0 0 0

Commit message: basic motion controller from coords

File: urdf/aplotter.urdf (robot description, URDF)
Before this commit: robot aplotter, 5 links, 4 joints
Joints:
- joint rightJoint: origin xyz=0 0 0 rpy=0 0 -0.12524034 -> xyz=0 0 0 rpy=0 0 0

Commit message: rviz2 mostly implemented

File: urdf/aplotter.urdf (robot description, URDF)
Before this commit: robot aplotter, 5 links, 4 joints
Joints:
- joint leftPJoint: origin xyz=0 41.356 71.042 rpy=0 0 0 -> xyz=0 0 71.042 rpy=0 0 0
- joint rightPJoint: origin xyz=0 41.356 71.042 rpy=0 0 0 -> xyz=0 0 71.042 rpy=0 0 0
